Commit message: update prj2

File: new_prj_2/src/my_robot/urdf/my_robot.xacro (robot description, xacro)
@@ -2,197 +2,190 @@
 <robot name="my_robot" xmlns:xacro="http://www.ros.org/wiki/xacro">
   <xacro:include filename="$(find my_robot)/urdf/my_robot.gazebo" />
-  <link name="robot_footprint"></link>
+  <link name="robot_footprint">
+  </link>
   <joint name="robot_footprint_joint" type="fixed">
     <origin xyz="0 0 0" rpy="0 0 0" />
-    <parent link="robot_footprint"/>
+    <parent link="robot_footprint" />
     <child link="chassis" />
   </joint>
   <link name='chassis'>
-    <pose>0 0 0.1 0 0 0</pose>
-    <inertial>
-      <mass value="15.0"/>
-      <origin xyz="0.0 0 0" rpy=" 0 0 0"/>
-      <inertia
-          ixx="0.1" ixy="0" ixz="0"
-          iyy="0.1" iyz="0"
-          izz="0.1"
-      />
-    </inertial>
-    <collision name='collision'>
-      <origin xyz="0 0 0" rpy=" 0 0 0"/>
-      <geometry>
-        <box size=".4 .2 .1"/>
-      </geometry>
-    </collision>
-    <visual name='chassis_visual'>
-      <origin xyz="0 0 0" rpy=" 0 0 0"/>
-      <geometry>
-        <box size=".4 .2 .1"/>
-      </geometry>
-    </visual>
-    <collision name='back_caster_collision'>
-      <origin xyz="-0.15 0 -0.05" rpy=" 0 0 0"/>
-      <geometry>
-        <sphere radius="0.0499"/>
-      </geometry>
-    </collision>
-    <visual name='back_caster_visual'>
-      <origin xyz="-0.15 0 -0.05" rpy=" 0 0 0"/>
-      <geometry>
-        <sphere radius="0.05"/>
-      </geometry>
-    </visual>
-    <collision name='front_caster_collision'>
-      <origin xyz="0.15 0 -0.05" rpy=" 0 0 0"/>
-      <geometry>
-        <sphere radius="0.0499"/>
-      </geometry>
-    </collision>
-    <visual name='front_caster_visual'>
-      <origin xyz="0.15 0 -0.05" rpy=" 0 0 0"/>
-      <geometry>
-        <sphere radius="0.05"/>
-      </geometry>
-    </visual>
+  <pose>0 0 0.1 0 0 0</pose>
+  <inertial>
+    <mass value="15.0" />
+    <origin xyz="0.0 0 0" rpy=" 0 0 0" />
+    <inertia ixx="0.1" ixy="0" ixz="0" iyy="0.1" iyz="0" izz="0.1" />
+  </inertial>
+  <collision name='collision'>
+    <origin xyz="0 0 0" rpy=" 0 0 0" />
+    <geometry>
+      <box size=".4 .2 .1" />
+    </geometry>
+  </collision>
+  <visual name='chassis_visual'>
+    <origin xyz="0 0 0" rpy=" 0 0 0" />
+    <geometry>
+      <box size=".4 .2 .1" />
+    </geometry>
+  </visual>
+  <collision name='back_caster_collision'>
+    <origin xyz="-0.15 0 -0.05" rpy=" 0 0 0" />
+    <geometry>
+      <sphere radius="0.0499" />
+    </geometry>
+  </collision>
+  <visual name='back_caster_visual'>
+    <origin xyz="-0.15 0 -0.05" rpy=" 0 0 0" />
+    <geometry>
+      <sphere radius="0.05" />
+    </geometry>
+  </visual>
+  <collision name='front_caster_collision'>
+    <origin xyz="0.15 0 -0.05" rpy=" 0 0 0" />
+    <geometry>
+      <sphere radius="0.0499" />
+    </geometry>
+  </collision>
+  <visual name='front_caster_visual'>
+    <origin xyz="0.15 0 -0.05" rpy=" 0 0 0" />
+    <geometry>
+      <sphere radius="0.05" />
+    </geometry>
+  </visual>
+    <collision name='top_caster_collision'>
+    <origin xyz="-0.1 0 0.08" rpy=" 0 0 0" />
+    <geometry>
+      <sphere radius="0.1" />
+    </geometry>
+  </collision>
+  <visual name='top_caster_visual'>
+    <origin xyz="-0.1 0 0.08" rpy=" 0 0 0" />
+    <geometry>
+      <sphere radius="0.1" />
+    </geometry>
+  </visual>
   </link>
   <!-- left wheel -->
   <joint type="continuous" name="left_wheel_hinge">
-    <origin xyz="0 0.15 0" rpy="0 0 0"/>
-    <child link="left_wheel"/>
-    <parent link="chassis"/>
-    <axis xyz="0 1 0" rpy="0 0 0"/>
-    <limit effort="10000" velocity="1000"/>
-    <dynamics damping="1.0" friction="1.0"/>
+    <origin xyz="0 0.15 0" rpy="0 0 0" />
+    <child link="left_wheel" />
+    <parent link="chassis" />
+    <axis xyz="0 1 0" rpy="0 0 0" />
+    <limit effort="10000" velocity="1000" />
+    <dynamics damping="1.0" friction="1.0" />
   </joint>
   <link name="left_wheel">
-    <inertial>
-      <mass value="5.0"/>
-      <origin xyz="0 0 0" rpy="0 1.5707 1.5707"/>
-      <inertia
-          ixx="0.1" ixy="0" ixz="0"
-          iyy="0.1" iyz="0"
-          izz="0.1"
-      />
-    </inertial>
-    <collision name='collision'>
-      <origin xyz="0 0 0" rpy=" 0 1.5707 1.5707"/>
-      <geometry>
-        <cylinder radius="0.1" length="0.05"/>
-      </geometry>
-    </collision>
-    <visual name="left_wheel_visual">
-        <origin xyz="0 0 0" rpy="0 1.5707 1.5707"/>
-        <geometry>
-            <cylinder radius="0.1" length="0.05"/>
-        </geometry>
-    </visual>
+  <inertial>
+    <mass value="5.0" />
+    <origin xyz="0 0 0" rpy="0 1.5707 1.5707" />
+    <inertia ixx="0.1" ixy="0" ixz="0" iyy="0.1" iyz="0" izz="0.1" />
+  </inertial>
+  <collision name='collision'>
+    <origin xyz="0 0 0" rpy=" 0 1.5707 1.5707" />
+    <geometry>
+      <cylinder radius="0.1" length="0.05" />
+    </geometry>
+  </collision>
+  <visual name="left_wheel_visual">
+    <origin xyz="0 0 0" rpy="0 1.5707 1.5707" />
+    <geometry>
+      <cylinder radius="0.1" length="0.05" />
+    </geometry>
+  </visual>
   </link>
   <!-- right wheel -->
   <joint type="continuous" name="right_wheel_hinge">
-    <origin xyz="0 -0.15 0" rpy="0 0 0"/>
-    <child link="right_wheel"/>
-    <parent link="chassis"/>
-    <axis xyz="0 1 0" rpy="0 0 0"/>
-    <limit effort="10000" velocity="1000"/>
-    <dynamics damping="1.0" friction="1.0"/>
+    <origin xyz="0 -0.15 0" rpy="0 0 0" />
+    <child link="right_wheel" />
+    <parent link="chassis" />
+    <axis xyz="0 1 0" rpy="0 0 0" />
+    <limit effort="10000" velocity="1000" />
+    <dynamics damping="1.0" friction="1.0" />
   </joint>
   <link name="right_wheel">
-    <inertial>
-      <mass value="5.0"/>
-      <origin xyz="0.0 0 0" rpy=" 0 1.5707 1.5707"/>
-      <inertia
-          ixx="0.1" ixy="0" ixz="0"
-          iyy="0.1" iyz="0"
-          izz="0.1"
-      />
-    </inertial>
-    <collision name='collision'>
-      <origin xyz="0 0 0" rpy=" 0 1.5707 1.5707"/>
-      <geometry>
-            <cylinder radius="0.1" length="0.05"/>
-      </geometry>
-    </collision>
-    <visual name="right_wheel_visual">
-        <origin xyz="0 0 0" rpy="0 1.5707 1.5707"/>
-        <geometry>
-            <cylinder radius="0.1" length="0.05"/>
-        </geometry>
-    </visual>
+  <inertial>
+    <mass value="5.0" />
+    <origin xyz="0.0 0 0" rpy=" 0 1.5707 1.5707" />
+    <inertia ixx="0.1" ixy="0" ixz="0" iyy="0.1" iyz="0" izz="0.1" />
+  </inertial>
+  <collision name='collision'>
+    <origin xyz="0 0 0" rpy=" 0 1.5707 1.5707" />
+    <geometry>
+      <cylinder radius="0.1" length="0.05" />
+    </geometry>
+  </collision>
+  <visual name="right_wheel_visual">
+    <origin xyz="0 0 0" rpy="0 1.5707 1.5707" />
+    <geometry>
+      <cylinder radius="0.1" length="0.05" />
+    </geometry>
+  </visual>
   </link>
   <!-- camera -->
   <link name="camera">
-    <inertial>
-      <mass value="0.1"/>
-      <origin xyz="0 0 0" rpy="0 0 0"/>
-      <inertia
-        ixx="1e-6" ixy="0" ixz="0"
-        iyy="1e-6" iyz="0"
-        izz="1e-6"
-      />
-    </inertial>
-    <collision name="collision">
-      <origin xyz="0 0 0" rpy="0 0 0"/>
-      <geometry>
-        <box size="0.05 0.05 0.05"/>
-      </geometry>
-    </collision>
-    <visual name="camera_visual">
-      <origin xyz="0 0 0" rpy="0 0 0"/>
-      <geometry>
-        <box size="0.05 0.05 0.05"/>
-      </geometry>
-    </visual>
+  <inertial>
+    <mass value="0.1" />
+    <origin xyz="0 0 0" rpy="0 0 0" />
+    <inertia ixx="1e-6" ixy="0" ixz="0" iyy="1e-6" iyz="0" izz="1e-6" />
+  </inertial>
+  <collision name="collision">
+    <origin xyz="0 0 0" rpy="0 0 0" />
+    <geometry>
+      <box size="0.05 0.05 0.05" />
+    </geometry>
+  </collision>
+  <visual name="camera_visual">
+    <origin xyz="0 0 0" rpy="0 0 0" />
+    <geometry>
+      <box size="0.05 0.05 0.05" />
+    </geometry>
+  </visual>
   </link>
   <joint type="fixed" name="camera_joint">
-    <origin xyz="0.2 0 0" rpy="0 0 0"/>
-    <child link="camera"/>
-    <parent link="chassis"/>
-    <axis xyz="0 1 0" rpy="0 0 0"/>
-    <limit effort="10000" velocity="1000"/>
-    <dynamics damping="1.0" friction="1.0"/>
+    <origin xyz="0.2 0 0" rpy="0 0 0" />
+    <child link="camera" />
+    <parent link="chassis" />
+    <axis xyz="0 1 0" rpy="0 0 0" />
+    <limit effort="10000" velocity="1000" />
+    <dynamics damping="1.0" friction="1.0" />
   </joint>
   <!-- lidar -->
   <link name="hokuyo">
-    <inertial>
-      <mass value="1e-5"/>
-      <origin xyz="0 0 0" rpy="0 0 0"/>
-      <inertia
-        ixx="1e-6" ixy="0" ixz="0"
-        iyy="1e-6" iyz="0"
-        izz="1e-6"
-      />
-    </inertial>
-    <collision name="collision">
-      <origin xyz="0 0 0" rpy="0 0 0"/>
-      <geometry>
-        <box size="0.1 0.1 0.1"/>
-      </geometry>
-    </collision>
-    <visual name="hokuyo_visual">
-      <origin xyz="0 0 0" rpy="0 0 0"/>
-      <geometry>
-        <mesh filename="package://my_robot/meshes/hokuyo.dae"/>
-      </geometry>
-    </visual>
+  <inertial>
+    <mass value="1e-5" />
+    <origin xyz="0 0 0" rpy="0 0 0" />
+    <inertia ixx="1e-6" ixy="0" ixz="0" iyy="1e-6" iyz="0" izz="1e-6" />
+  </inertial>
+  <collision name="collision">
+    <origin xyz="0 0 0" rpy="0 0 0" />
+    <geometry>
+      <box size="0.1 0.1 0.1" />
+    </geometry>
+  </collision>
+  <visual name="hokuyo_visual">
+    <origin xyz="0 0 0" rpy="0 0 0" />
+    <geometry>
+      <mesh filename="package://my_robot/meshes/hokuyo.dae" />
+    </geometry>
+  </visual>
   </link>
   <joint type="fixed" name="hokuyo_joint">
-    <origin xyz="0.15 0 0.1" rpy="0 0 0"/>
-    <child link="hokuyo"/>
-    <parent link="chassis"/>
-    <axis xyz="0 1 0" rpy="0 0 0"/>
-    <limit effort="10000" velocity="1000"/>
-    <dynamics damping="1.0" friction="1.0"/>
+    <origin xyz="0.15 0 0.1" rpy="0 0 0" />
+    <child link="hokuyo" />
+    <parent link="chassis" />
+    <axis xyz="0 1 0" rpy="0 0 0" />
+    <limit effort="10000" velocity="1000" />
+    <dynamics damping="1.0" friction="1.0" />
   </joint>
   <gazebo reference="left_wheel">
+    <material>Gazebo/Black</material>
+  </gazebo>
+  <gazebo reference="right_wheel">
+    <material>Gazebo/Black</material>
+  </gazebo>
+  <gazebo reference="chassis">
+    <material>Gazebo/Orange</material>
+  </gazebo>
+  <gazebo reference="camera">
     <material>Gazebo/Green</material>
   </gazebo>
-  <gazebo reference="right_wheel">
-    <material>Gazebo/Green</material>
-  </gazebo>
-  <gazebo reference="chassis">
-    <material>Gazebo/Blue</material>
-  </gazebo>
-  <gazebo reference="camera">
-    <material>Gazebo/Red</material>
-  </gazebo>
 </robot>
