Commit message: update project files

File: map_my_world/src/my_robot/urdf/my_robot.xacro (robot description, xacro)
@@ -123,5 +123,5 @@
   </link>
   <!-- camera -->
-  <!-- <link name="camera">
+  <link name="camera">
     <inertial>
       <mass value="0.1" />
@@ -143,5 +143,5 @@
   </link>
   <joint type="fixed" name="camera_joint">
-    <origin xyz="0.2 0 -0.03" rpy="0 0 0" />
+    <origin xyz="0.2 0 0" rpy="0 0 0" />
     <child link="camera" />
     <parent link="chassis" />
@@ -149,28 +149,11 @@
     <limit effort="10000" velocity="1000" />
     <dynamics damping="1.0" friction="1.0" />
-  </joint> -->
+  </joint>
   <!-- RGB-D camera -->
   <link name="camera_link_optical">
-    <inertial>
-      <mass value="0.1" />
-      <origin xyz="0 0 0" rpy="0 0 0" />
-      <inertia ixx="1e-6" ixy="0" ixz="0" iyy="1e-6" iyz="0" izz="1e-6" />
-    </inertial>
-    <collision name="collision">
-      <origin xyz="0 0 0" rpy="0 0 0" />
-      <geometry>
-        <box size="0.05 0.05 0.05" />
-      </geometry>
-    </collision>
-    <visual name="camera_visual">
-      <origin xyz="0 0 0" rpy="0 0 0" />
-      <geometry>
-        <box size="0.05 0.05 0.05" />
-      </geometry>
-    </visual>
   </link>
   <joint name="camera_optical_joint" type="fixed">
-    <origin xyz="0.2 0 0" rpy="0 0 0"/>
-    <parent link="chassis"/>
+    <origin xyz="0 0 0" rpy="0 0 0"/>
+    <parent link="camera"/>
     <child link="camera_link_optical"/>
     <axis xyz="0 1 0" rpy="0 0 0" />

Commit message: update mapping project.

File: map_my_world/src/my_robot/urdf/my_robot.xacro (robot description, xacro)
@@ -154,5 +154,5 @@
   </link>
   <joint name="camera_optical_joint" type="fixed">
-    <origin xyz="0 0 0" rpy="0 0 0"/>
+    <origin xyz="0 0 0" rpy="-1.5707 0 -1.5707"/>
     <parent link="camera"/>
     <child link="camera_link_optical"/>
